Commit message: implement the gripper (no physic yet)

File: urdf/link_joint.xacro (robot description, xacro)
@@ -41,4 +41,24 @@
         </link>
     </xacro:macro>
+    <xacro:macro name="xacro_mesh" params="name file origin_rpy origin_xyz mass scale">
+        <link name="${name}">
+            <visual>
+                <geometry>
+                    <mesh filename="${file}" scale="${scale} ${scale} ${scale}"/>
+                </geometry>
+                <origin rpy="${origin_rpy}" xyz="${origin_xyz}"/>
+            </visual>
+            <collision>
+                <geometry>
+                    <mesh filename="${file}" scale="${scale} ${scale} ${scale}"/>
+                </geometry>
+                <origin rpy="${origin_rpy}" xyz="${origin_xyz}"/>
+            </collision>
+            <inertial>
+                <mass value="${mass}"/>
+                <inertia ixx="0.01" ixy="0.0" ixz="0.0" iyy="0.01" iyz="0.0" izz="0.01"/>
+            </inertial>
+        </link>
+    </xacro:macro>
     <xacro:macro name="xacro_joint" params="name type axis lower upper parent child origin_xyz">
         <joint name="${name}" type="${type}">

File: urdf/model1.xacro (robot description, xacro)
@@ -107,3 +107,49 @@
         joint="arm2_arm3_joint"
     />
+    <xacro:xacro_mesh
+        name="gripper1"
+        file="package://urdf1/mesh/gripper1.dae"
+        origin_rpy="1.57 0 1.57"
+        origin_xyz="-0.15 0 0"
+        mass="0.1"
+        scale="3"
+    />
+    <xacro:xacro_joint
+        name="arm3_gripper1_joint"
+        type="revolute"
+        axis="-1 0 0"
+        lower="-3.14"
+        upper="0"
+        parent="arm3"
+        child="gripper1"
+        origin_xyz="0 0 0.5"
+    />
+    <xacro:xacro_trans_position
+        name="arm3_gripper1_trans"
+        actuator="arm3_gripper1_actuator"
+        joint="arm3_gripper1_joint"
+    />
+    <xacro:xacro_mesh
+        name="gripper2"
+        file="package://urdf1/mesh/gripper2.dae"
+        origin_rpy="1.57 0 1.57"
+        origin_xyz="-0.15 0 0"
+        mass="0.1"
+        scale="3"
+    />
+    <xacro:xacro_joint
+        name="arm3_gripper2_joint"
+        type="revolute"
+        axis="1 0 0"
+        lower="-3.14"
+        upper="0"
+        parent="arm3"
+        child="gripper2"
+        origin_xyz="0 0 0.5"
+    />
+    <xacro:xacro_trans_position
+        name="arm3_gripper2_trans"
+        actuator="arm3_gripper2_actuator"
+        joint="arm3_gripper2_joint"
+    />
 </robot>
