Commit message: add PID

File: urdf/model1.xacro (robot description, xacro)
@@ -26,4 +26,5 @@
         type="revolute"
         axis="0 0 1"
+        effort="1000"
         lower="-3.14"
         upper="3.14"
@@ -51,4 +52,5 @@
         type="revolute"
         axis="0 1 0"
+        effort="1000"
         lower="-3.14"
         upper="3.14"
@@ -76,4 +78,5 @@
         type="revolute"
         axis="0 1 0"
+        effort="1000"
         lower="-3.14"
         upper="3.14"
@@ -101,4 +104,5 @@
         type="revolute"
         axis="0 1 0"
+        effort="1000"
         lower="-3.14"
         upper="3.14"
@@ -125,4 +129,5 @@
         type="revolute"
         axis="-1 0 0"
+        effort="10"
         lower="-3.14"
         upper="0"
@@ -149,4 +154,5 @@
         type="revolute"
         axis="1 0 0"
+        effort="10"
         lower="-3.14"
         upper="0"

File: urdf/xacro/link_joint.xacro (robot description, xacro)
@@ -90,8 +90,8 @@
         </link>
     </xacro:macro>
-    <xacro:macro name="xacro_joint" params="name type axis lower upper parent child origin_xyz">
+    <xacro:macro name="xacro_joint" params="name type axis effort lower upper parent child origin_xyz">
         <joint name="${name}" type="${type}">
             <axis xyz="${axis}"/>
-            <limit effort="1000.0" lower="${lower}" upper="${upper}" velocity="0.5"/>
+            <limit effort="${effort}" lower="${lower}" upper="${upper}" velocity="0.5"/>
             <parent link="${parent}"/>
             <child link="${child}"/>

File: urdf/xacro/transmission.xacro (robot description, xacro)
@@ -7,4 +7,7 @@
 		    </type>
 		    <actuator name="${actuator}">
+                <hardwareInterface>
+                    hardware_interface/EffortJointInterface
+                </hardwareInterface>
 		    	<mechanicalReduction>
 		    		1
@@ -13,5 +16,5 @@
             <joint name="${joint}">
                 <hardwareInterface>
-                    hardware_interface/PositionJointInterface
+                    hardware_interface/EffortJointInterface
                 </hardwareInterface>
             </joint>

Commit message: fix bounce (add damping+friction at all joints)

File: urdf/model1.xacro (robot description, xacro)
@@ -26,10 +26,9 @@
         type="revolute"
         axis="0 0 1"
-        effort="1000"
         lower="-3.14"
         upper="3.14"
         parent="stationary_base"
         child="spin_base"
-        origin_xyz="0 0 0.05"
+        origin_xyz="0 0 0.06"
     />
     <xacro:xacro_trans_position
@@ -52,10 +51,9 @@
         type="revolute"
         axis="0 1 0"
-        effort="1000"
-        lower="-3.14"
-        upper="3.14"
+        lower="-1.57"
+        upper="1.57"
         parent="spin_base"
         child="arm1"
-        origin_xyz="0 0 0.05"
+        origin_xyz="0 0 0.2"
     />
     <xacro:xacro_trans_position
@@ -71,5 +69,5 @@
         d="0.1"
         origin_rpy="0 1.57 0"
-        origin_xyz="0 0 0.5"
+        origin_xyz="0 0.05 0.5"
         mass="0.5"
     />
@@ -78,10 +76,9 @@
         type="revolute"
         axis="0 1 0"
-        effort="1000"
         lower="-3.14"
         upper="3.14"
         parent="arm1"
         child="arm2"
-        origin_xyz="0 0 1"
+        origin_xyz="0 0.05 1"
     />
     <xacro:xacro_trans_position
@@ -97,5 +94,5 @@
         d="0.1"
         origin_rpy="0 1.57 0"
-        origin_xyz="0 0 0.25"
+        origin_xyz="0 -0.05 0.25"
         mass="0.5"
     />
@@ -104,5 +101,4 @@
         type="revolute"
         axis="0 1 0"
-        effort="1000"
         lower="-3.14"
         upper="3.14"
@@ -129,10 +125,9 @@
         type="revolute"
         axis="-1 0 0"
-        effort="10"
         lower="-3.14"
         upper="0"
         parent="arm3"
         child="gripper1"
-        origin_xyz="0 0 0.5"
+        origin_xyz="0 -0.05 0.5"
     />
     <xacro:xacro_trans_position
@@ -154,10 +149,9 @@
         type="revolute"
         axis="1 0 0"
-        effort="10"
         lower="-3.14"
         upper="0"
         parent="arm3"
         child="gripper2"
-        origin_xyz="0 0 0.5"
+        origin_xyz="0 -0.05 0.5"
     />
     <xacro:xacro_trans_position

File: urdf/xacro/link_joint.xacro (robot description, xacro)
@@ -21,5 +21,5 @@
                     </friction>
                     <torsional>
-                        <coefficient>2.0</coefficient>
+                        <coefficient>1</coefficient>
                         <surface_radius>0.5</surface_radius>
                         <use_patch_radius>false</use_patch_radius>
@@ -90,11 +90,12 @@
         </link>
     </xacro:macro>
-    <xacro:macro name="xacro_joint" params="name type axis effort lower upper parent child origin_xyz">
+    <xacro:macro name="xacro_joint" params="name type axis lower upper parent child origin_xyz">
         <joint name="${name}" type="${type}">
             <axis xyz="${axis}"/>
-            <limit effort="${effort}" lower="${lower}" upper="${upper}" velocity="0.5"/>
+            <limit effort="100" lower="${lower}" upper="${upper}" velocity="1"/>
             <parent link="${parent}"/>
             <child link="${child}"/>
             <origin xyz="${origin_xyz}"/>
+            <dynamics damping="10.0" friction="0.3"/> <!-- very very important -->
         </joint>
     </xacro:macro>

Commit message: change package name to robotarm and fix gripper

File: urdf/model1.xacro (robot description, xacro)
@@ -1,7 +1,13 @@
 <?xml version="1.0"?>
 <robot name="robotarm" xmlns:xacro="http://www.ros.org/wiki/xacro">
-    <xacro:include filename="$(find urdf1)/urdf/xacro/link_joint.xacro"/>
-    <xacro:include filename="$(find urdf1)/urdf/xacro/transmission.xacro"/>
-    <xacro:include filename="$(find urdf1)/urdf/xacro/gazebo.xacro"/>
+    <xacro:include filename="$(find robotarm)/urdf/xacro/link_joint.xacro"/>
+    <xacro:include filename="$(find robotarm)/urdf/xacro/transmission.xacro"/>
+    <xacro:include filename="$(find robotarm)/urdf/xacro/gazebo.xacro"/>
+    <!-- fix model to world -->
+    <link name="world"/>
+    <joint name="fixed" type="fixed">
+        <parent link="world"/>
+        <child link="stationary_base"/>
+    </joint>
     <!-- stationary_base -->
     <xacro:xacro_cylinder
@@ -115,5 +121,5 @@
     <xacro:xacro_mesh
         name="gripper1"
-        file="package://urdf1/mesh/gripper1.dae"
+        file="package://robotarm/mesh/gripper1.dae"
         origin_rpy="1.57 0 1.57"
         origin_xyz="-0.15 0 0"
@@ -139,5 +145,5 @@
     <xacro:xacro_mesh
         name="gripper2"
-        file="package://urdf1/mesh/gripper2.dae"
+        file="package://robotarm/mesh/gripper2.dae"
         origin_rpy="1.57 0 1.57"
         origin_xyz="-0.15 0 0"

File: urdf/xacro/link_joint.xacro (robot description, xacro)
@@ -16,11 +16,11 @@
                     <friction>
                         <ode>
-                            <mu>0.1</mu>
-                            <mu2>0.1</mu2>
+                            <mu>0.5</mu>
+                            <mu2>0.5</mu2>
                         </ode>
                     </friction>
                     <torsional>
                         <coefficient>1</coefficient>
-                        <surface_radius>0.5</surface_radius>
+                        <surface_radius>1</surface_radius>
                         <use_patch_radius>false</use_patch_radius>
                     </torsional>
@@ -49,6 +49,6 @@
                     <friction>
                         <ode>
-                            <mu>0.1</mu>
-                            <mu2>0.1</mu2>
+                            <mu>0.5</mu>
+                            <mu2>0.5</mu2>
                         </ode>
                     </friction>
@@ -77,6 +77,6 @@
                     <friction>
                         <ode>
-                            <mu>0.1</mu>
-                            <mu2>0.1</mu2>
+                            <mu>0.8</mu>
+                            <mu2>0.8</mu2>
                         </ode>
                     </friction>
@@ -93,5 +93,5 @@
         <joint name="${name}" type="${type}">
             <axis xyz="${axis}"/>
-            <limit effort="100" lower="${lower}" upper="${upper}" velocity="1"/>
+            <limit effort="100" lower="${lower}" upper="${upper}" velocity="2"/>
             <parent link="${parent}"/>
             <child link="${child}"/>
