Commit message: add gazebo element to urdf file

File: urdf/xacro/gazebo.xacro (robot description, xacro)
@@ -6,3 +6,52 @@
         </plugin>
     </gazebo>
+    <!-- stationary_base -->
+    <gazebo reference="stationary_base">
+        <gravity>true</gravity>
+        <mu1>0.2</mu1>
+        <mu2>0.2</mu2>
+        <selfCollide>true</selfCollide>
+    </gazebo>
+    <!-- spin_base -->
+    <gazebo reference="spin_base">
+        <gravity>true</gravity>
+        <mu1>0.2</mu1>
+        <mu2>0.2</mu2>
+        <selfCollide>true</selfCollide>
+    </gazebo>
+    <!-- arm1 -->
+    <gazebo reference="arm1">
+        <gravity>true</gravity>
+        <mu1>0.2</mu1>
+        <mu2>0.2</mu2>
+        <selfCollide>true</selfCollide>
+    </gazebo>
+    <!-- arm2 -->
+    <gazebo reference="arm2">
+        <gravity>true</gravity>
+        <mu1>0.2</mu1>
+        <mu2>0.2</mu2>
+        <selfCollide>true</selfCollide>
+    </gazebo>
+    <!-- arm3 -->
+    <gazebo reference="arm3">
+        <gravity>true</gravity>
+        <mu1>0.2</mu1>
+        <mu2>0.2</mu2>
+        <selfCollide>true</selfCollide>
+    </gazebo>
+    <!-- gripper1 -->
+    <gazebo reference="gripper1">
+        <gravity>true</gravity>
+        <mu1>0.2</mu1>
+        <mu2>0.2</mu2>
+        <selfCollide>true</selfCollide>
+    </gazebo>
+    <!-- gripper2 -->
+    <gazebo reference="gripper2">
+        <gravity>true</gravity>
+        <mu1>0.2</mu1>
+        <mu2>0.2</mu2>
+        <selfCollide>true</selfCollide>
+    </gazebo>
 </robot>

File: urdf/xacro/link_joint.xacro (robot description, xacro)
@@ -97,5 +97,5 @@
             <child link="${child}"/>
             <origin xyz="${origin_xyz}"/>
-            <dynamics damping="10.0" friction="0.3"/> <!-- very very important -->
+            <dynamics damping="10.0" friction="0.3"/>
         </joint>
     </xacro:macro>
